File: eagle/sch.brd (EAGLE design)
At the start: 151.1 x 100 mm, 28 parts, among them IC1 MEGA32-P, T1 2N2222, T2 2N2222

Commit message: keypad
Parts:
- added S1, S10, S11, S12, S13, S14, S15, S16, S2, S3, S4, S5, S6, S7, S8, S9: DTS-3, switch-tact:DTS-3
- added SW5: (no value), special:EDG-08
Connections:
- new net A0: IC1.40, SW5.8
- new net A1: IC1.39, SW5.7
- new net A2: IC1.38, SW5.6
- new net A3: IC1.37, SW5.5
- new net A4: IC1.36, SW5.4
- new net A5: IC1.35, SW5.3
- new net A6: IC1.34, SW5.2
- new net A7: IC1.33, SW5.1
- new net N$12: S1.2, S13.2, S5.2, S9.2, SW5.13
- new net N$27: S10.2, S14.2, S2.2, S6.2, SW5.14
- new net N$30: S11.2, S15.2, S3.2, S7.2, SW5.15
- new net N$31: S1.1, S2.1, S3.1, S4.1, SW5.9
- new net N$34: S12.2, S16.2, S4.2, S8.2, SW5.16
- new net N$41: S5.1, S6.1, S7.1, S8.1, SW5.10
- new net N$49: S10.1, S11.1, S12.1, S9.1, SW5.11
- new net N$57: S13.1, S14.1, S15.1, S16.1, SW5.12
Changed lines of the file:
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@@
 <attribute name="PROD_ID" value="RES-09327" x="54.61" y="64.77" size="1.778" layer="27" display="off"/>
 </element>
+<element name="S1" library="switch-tact" package="DTS-3" value="DTS-3" x="96.52" y="93.98"/>
+<element name="SW5" library="special" library_urn="urn:adsk.eagle:library:367" package="EDG-08" package3d_urn="urn:adsk.eagle:package:26659/2" value="" x="73.66" y="85.09" rot="MR90"/>
+<element name="S2" library="switch-tact" package="DTS-3" value="DTS-3" x="111.76" y="93.98"/>
+<element name="S3" library="switch-tact" package="DTS-3" value="DTS-3" x="127" y="93.98"/>
+<element name="S4" library="switch-tact" package="DTS-3" value="DTS-3" x="142.24" y="93.98"/>
+<element name="S5" library="switch-tact" package="DTS-3" value="DTS-3" x="96.52" y="87.63"/>
+<element name="S6" library="switch-tact" package="DTS-3" value="DTS-3" x="111.76" y="87.63"/>
+<element name="S7" library="switch-tact" package="DTS-3" value="DTS-3" x="127" y="87.63"/>
+<element name="S8" library="switch-tact" package="DTS-3" value="DTS-3" x="142.24" y="87.63"/>
+<element name="S9" library="switch-tact" package="DTS-3" value="DTS-3" x="96.52" y="81.28"/>
+<element name="S10" library="switch-tact" package="DTS-3" value="DTS-3" x="111.76" y="81.28"/>
+<element name="S11" library="switch-tact" package="DTS-3" value="DTS-3" x="127" y="81.28"/>
+<element name="S12" library="switch-tact" package="DTS-3" value="DTS-3" x="142.24" y="81.28"/>
+<element name="S13" library="switch-tact" package="DTS-3" value="DTS-3" x="96.52" y="74.93"/>
+<element name="S14" library="switch-tact" package="DTS-3" value="DTS-3" x="111.76" y="74.93"/>
+<element name="S15" library="switch-tact" package="DTS-3" value="DTS-3" x="127" y="74.93"/>
+<element name="S16" library="switch-tact" package="DTS-3" value="DTS-3" x="142.24" y="74.93"/>
 </elements>
 <signals>
@@
 <contactref element="T2" pad="C"/>
 <contactref element="T1" pad="C"/>
-<wire x1="41.91" y1="68.58" x2="40.64" y2="49.53" width="0" layer="19" extent="1-1"/>
+<wire x1="40.64" y1="49.53" x2="41.91" y2="68.58" width="0" layer="19" extent="1-1"/>
 <wire x1="55.88" y1="25.4" x2="40.64" y2="49.53" width="0" layer="19" extent="1-1"/>
 <wire x1="17.78" y1="25.4" x2="40.64" y2="49.53" width="0" layer="19" extent="1-1"/>
@@
 <wire x1="58.42" y1="68.58" x2="43.18" y2="58.42" width="0" layer="19" extent="1-1"/>
 </signal>
+<signal name="A7">
+<contactref element="IC1" pad="33"/>
+<contactref element="SW5" pad="1"/>
+<wire x1="68.58" y1="57.15" x2="69.85" y2="76.2" width="0" layer="19" extent="1-1"/>
+</signal>
+<signal name="A6">
+<contactref element="IC1" pad="34"/>
+<contactref element="SW5" pad="2"/>
+<wire x1="66.04" y1="57.15" x2="69.85" y2="78.74" width="0" layer="19" extent="1-1"/>
+</signal>
+<signal name="A5">
+<contactref element="IC1" pad="35"/>
+<contactref element="SW5" pad="3"/>
+<wire x1="63.5" y1="57.15" x2="69.85" y2="81.28" width="0" layer="19" extent="1-1"/>
+</signal>
+<signal name="A4">
+<contactref element="IC1" pad="36"/>
+<contactref element="SW5" pad="4"/>
+<wire x1="60.96" y1="57.15" x2="69.85" y2="83.82" width="0" layer="19" extent="1-1"/>
+</signal>
+<signal name="A3">
+<contactref element="IC1" pad="37"/>
+<contactref element="SW5" pad="5"/>
+<wire x1="58.42" y1="57.15" x2="69.85" y2="86.36" width="0" layer="19" extent="1-1"/>
+</signal>
+<signal name="A2">
+<contactref element="IC1" pad="38"/>
+<contactref element="SW5" pad="6"/>
+<wire x1="55.88" y1="57.15" x2="69.85" y2="88.9" width="0" layer="19" extent="1-1"/>
+</signal>
+<signal name="A1">
+<contactref element="IC1" pad="39"/>
+<contactref element="SW5" pad="7"/>
+<wire x1="53.34" y1="57.15" x2="69.85" y2="91.44" width="0" layer="19" extent="1-1"/>
+</signal>
+<signal name="A0">
+<contactref element="IC1" pad="40"/>
+<contactref element="SW5" pad="8"/>
+<wire x1="50.8" y1="57.15" x2="69.85" y2="93.98" width="0" layer="19" extent="1-1"/>
+</signal>
+<signal name="N$12">
+<contactref element="S1" pad="2"/>
+<contactref element="S5" pad="2"/>
+<contactref element="S9" pad="2"/>
+<contactref element="S13" pad="2"/>
+<contactref element="SW5" pad="13"/>
+<wire x1="99.77" y1="87.63" x2="99.77" y2="81.28" width="0" layer="19" extent="1-1"/>
+<wire x1="99.77" y1="74.93" x2="99.77" y2="81.28" width="0" layer="19" extent="1-1"/>
+<wire x1="77.47" y1="83.82" x2="99.77" y2="87.63" width="0" layer="19" extent="1-1"/>
+<wire x1="99.77" y1="93.98" x2="77.47" y2="83.82" width="0" layer="19" extent="1-1"/>
+</signal>
+<signal name="N$27">
+<contactref element="S2" pad="2"/>
+<contactref element="S6" pad="2"/>
+<contactref element="S10" pad="2"/>
+<contactref element="S14" pad="2"/>
+<contactref element="SW5" pad="14"/>
+<wire x1="115.01" y1="87.63" x2="115.01" y2="81.28" width="0" layer="19" extent="1-1"/>
+<wire x1="115.01" y1="93.98" x2="115.01" y2="87.63" width="0" layer="19" extent="1-1"/>
+<wire x1="77.47" y1="81.28" x2="115.01" y2="93.98" width="0" layer="19" extent="1-1"/>
+<wire x1="115.01" y1="74.93" x2="115.01" y2="81.28" width="0" layer="19" extent="1-1"/>
+</signal>
+<signal name="N$30">
+<contactref element="S3" pad="2"/>
+<contactref element="S7" pad="2"/>
+<contactref element="S11" pad="2"/>
+<contactref element="S15" pad="2"/>
+<contactref element="SW5" pad="15"/>
+<wire x1="130.25" y1="93.98" x2="130.25" y2="87.63" width="0" layer="19" extent="1-1"/>
+<wire x1="77.47" y1="78.74" x2="130.25" y2="93.98" width="0" layer="19" extent="1-1"/>
+<wire x1="130.25" y1="81.28" x2="130.25" y2="87.63" width="0" layer="19" extent="1-1"/>
+<wire x1="130.25" y1="74.93" x2="130.25" y2="81.28" width="0" layer="19" extent="1-1"/>
+</signal>
+<signal name="N$31">
+<contactref element="S4" pad="1"/>
+<contactref element="S3" pad="1"/>
+<contactref element="S2" pad="1"/>
+<contactref element="S1" pad="1"/>
+<contactref element="SW5" pad="9"/>
+<wire x1="77.47" y1="93.98" x2="93.27" y2="93.98" width="0" layer="19" extent="1-1"/>
+<wire x1="108.51" y1="93.98" x2="77.47" y2="93.98" width="0" layer="19" extent="1-1"/>
+<wire x1="123.75" y1="93.98" x2="108.51" y2="93.98" width="0" layer="19" extent="1-1"/>
+<wire x1="138.99" y1="93.98" x2="123.75" y2="93.98" width="0" layer="19" extent="1-1"/>
+</signal>
+<signal name="N$34">
+<contactref element="S4" pad="2"/>
+<contactref element="S8" pad="2"/>
+<contactref element="S12" pad="2"/>
+<contactref element="S16" pad="2"/>
+<contactref element="SW5" pad="16"/>
+<wire x1="145.49" y1="93.98" x2="145.49" y2="87.63" width="0" layer="19" extent="1-1"/>
+<wire x1="77.47" y1="76.2" x2="145.49" y2="93.98" width="0" layer="19" extent="1-1"/>
+<wire x1="145.49" y1="81.28" x2="145.49" y2="87.63" width="0" layer="19" extent="1-1"/>
+<wire x1="145.49" y1="74.93" x2="145.49" y2="81.28" width="0" layer="19" extent="1-1"/>
+</signal>
+<signal name="N$41">
+<contactref element="S8" pad="1"/>
+<contactref element="S7" pad="1"/>
+<contactref element="S6" pad="1"/>
+<contactref element="S5" pad="1"/>
+<contactref element="SW5" pad="10"/>
+<wire x1="123.75" y1="87.63" x2="138.99" y2="87.63" width="0" layer="19" extent="1-1"/>
+<wire x1="108.51" y1="87.63" x2="123.75" y2="87.63" width="0" layer="19" extent="1-1"/>
+<wire x1="93.27" y1="87.63" x2="108.51" y2="87.63" width="0" layer="19" extent="1-1"/>
+<wire x1="77.47" y1="91.44" x2="93.27" y2="87.63" width="0" layer="19" extent="1-1"/>
+</signal>
+<signal name="N$49">
+<contactref element="S12" pad="1"/>
+<contactref element="S11" pad="1"/>
+<contactref element="S10" pad="1"/>
+<contactref element="S9" pad="1"/>
+<contactref element="SW5" pad="11"/>
+<wire x1="93.27" y1="81.28" x2="108.51" y2="81.28" width="0" layer="19" extent="1-1"/>
+<wire x1="123.75" y1="81.28" x2="108.51" y2="81.28" width="0" layer="19" extent="1-1"/>
+<wire x1="138.99" y1="81.28" x2="123.75" y2="81.28" width="0" layer="19" extent="1-1"/>
+<wire x1="77.47" y1="88.9" x2="93.27" y2="81.28" width="0" layer="19" extent="1-1"/>
+</signal>
+<signal name="N$57">
+<contactref element="S16" pad="1"/>
+<contactref element="S15" pad="1"/>
+<contactref element="S14" pad="1"/>
+<contactref element="S13" pad="1"/>
+<contactref element="SW5" pad="12"/>
+<wire x1="123.75" y1="74.93" x2="138.99" y2="74.93" width="0" layer="19" extent="1-1"/>
+<wire x1="108.51" y1="74.93" x2="123.75" y2="74.93" width="0" layer="19" extent="1-1"/>
+<wire x1="93.27" y1="74.93" x2="108.51" y2="74.93" width="0" layer="19" extent="1-1"/>
+<wire x1="77.47" y1="86.36" x2="93.27" y2="74.93" width="0" layer="19" extent="1-1"/>
+</signal>
 </signals>

Commit message: ADC
Parts:
- added ANALOG, ANALOG1: (no value), special:EDG-01
- added POT2: (no value), pot:B25P
Connections:
- new net N$29: ANALOG1.2, POT2.S
- net 5V: now also ANALOG.2, POT2.E
- net A0: now also ANALOG1.1
- net AVCC: now also ANALOG.1
- net GND: now also POT2.A
Changed lines of the file:
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@@
 <element name="S15" library="switch-tact" package="DTS-3" value="DTS-3" x="127" y="74.93"/>
 <element name="S16" library="switch-tact" package="DTS-3" value="DTS-3" x="142.24" y="74.93"/>
+<element name="ANALOG" library="special" library_urn="urn:adsk.eagle:library:367" package="EDG-01" package3d_urn="urn:adsk.eagle:package:26661/1" value="" x="76.2" y="64.77"/>
+<element name="POT2" library="pot" package="B25P" value="" x="43.18" y="92.71"/>
+<element name="ANALOG1" library="special" library_urn="urn:adsk.eagle:library:367" package="EDG-01" package3d_urn="urn:adsk.eagle:package:26661/1" value="" x="50.8" y="91.44"/>
 </elements>
 <signals>
-<signal name="AVCC">
-<contactref element="IC1" pad="30"/>
-</signal>
 <signal name="VCC">
 <contactref element="IC1" pad="10"/>
@@
 <contactref element="J1" pad="1"/>
 <contactref element="POT1" pad="A"/>
-<wire x1="123.19" y1="5.08" x2="7.62" y2="21.59" width="0" layer="19" extent="1-1"/>
-<wire x1="107.95" y1="5.08" x2="123.19" y2="5.08" width="0" layer="19" extent="1-1"/>
-<wire x1="76.2" y1="41.91" x2="107.95" y2="5.08" width="0" layer="19" extent="1-1"/>
-<wire x1="73.66" y1="57.15" x2="76.2" y2="41.91" width="0" layer="19" extent="1-1"/>
+<contactref element="POT2" pad="A"/>
+<wire x1="76.2" y1="41.91" x2="73.66" y2="57.15" width="0" layer="19" extent="1-1"/>
 <wire x1="50.55" y1="10.42" x2="76.2" y2="41.91" width="0" layer="19" extent="1-1"/>
 <wire x1="50.8" y1="10.16" x2="50.55" y2="10.42" width="0" layer="19" extent="1-1"/>
 <wire x1="12.7" y1="10.16" x2="50.55" y2="10.42" width="0" layer="19" extent="1-1"/>
 <wire x1="12.45" y1="10.42" x2="12.7" y2="10.16" width="0" layer="19" extent="1-1"/>
+<wire x1="7.62" y1="21.59" x2="12.45" y2="10.42" width="0" layer="19" extent="1-1"/>
+<wire x1="107.95" y1="5.08" x2="76.2" y2="41.91" width="0" layer="19" extent="1-1"/>
+<wire x1="123.19" y1="5.08" x2="107.95" y2="5.08" width="0" layer="19" extent="1-1"/>
+<wire x1="40.64" y1="92.71" x2="12.7" y2="10.16" width="0" layer="19" extent="1-1"/>
 </signal>
 <signal name="D0">
@@
 <contactref element="T2" pad="C"/>
 <contactref element="T1" pad="C"/>
+<contactref element="ANALOG" pad="2"/>
+<contactref element="POT2" pad="E"/>
+<wire x1="41.91" y1="68.58" x2="76.2" y2="68.58" width="0" layer="19" extent="1-1"/>
 <wire x1="40.64" y1="49.53" x2="41.91" y2="68.58" width="0" layer="19" extent="1-1"/>
 <wire x1="55.88" y1="25.4" x2="40.64" y2="49.53" width="0" layer="19" extent="1-1"/>
 <wire x1="17.78" y1="25.4" x2="40.64" y2="49.53" width="0" layer="19" extent="1-1"/>
 <wire x1="12.7" y1="21.59" x2="17.78" y2="25.4" width="0" layer="19" extent="1-1"/>
+<wire x1="45.72" y1="92.71" x2="12.7" y2="21.59" width="0" layer="19" extent="1-1"/>
 </signal>
 <signal name="C0">
@@
 <contactref element="IC1" pad="40"/>
 <contactref element="SW5" pad="8"/>
+<contactref element="ANALOG1" pad="1"/>
 <wire x1="50.8" y1="57.15" x2="69.85" y2="93.98" width="0" layer="19" extent="1-1"/>
+<wire x1="50.8" y1="87.63" x2="50.8" y2="57.15" width="0" layer="19" extent="1-1"/>
 </signal>
 <signal name="N$12">
@@
 <wire x1="77.47" y1="86.36" x2="93.27" y2="74.93" width="0" layer="19" extent="1-1"/>
 </signal>
+<signal name="AVCC">
+<contactref element="IC1" pad="30"/>
+<contactref element="ANALOG" pad="1"/>
+<wire x1="76.2" y1="60.96" x2="76.2" y2="57.15" width="0" layer="19" extent="1-1"/>
+</signal>
+<signal name="N$29">
+<contactref element="POT2" pad="S"/>
+<contactref element="ANALOG1" pad="2"/>
+<wire x1="43.18" y1="95.25" x2="50.8" y2="95.25" width="0" layer="19" extent="1-1"/>
+</signal>
 </signals>

Commit message: sch_001
Parts:
- removed ANALOG1: (no value), special:EDG-01
- added A: (no value), special:EDG-01
- added D1: 1N4446, diode:DO35-10
- added IC2: (no value), v-reg:78MXXL
- added J2: (no value), con-jack:SPC4077
- added LED9: (no value), led:LED5MM
- added PORTA, PORTB, PORTC, PORTD: (no value), con-lstb:MA10-1
- added Q1: (no value), crystal:HC49U-V
- added R7: 10M, SparkFun-Resistors:AXIAL-0.3
- added SV1: (no value), con-lstb:MA03-1
- moved U$1 115.9 mm to (90.2, 25.4), turned to 90 degrees
- moved R4 43.3 mm to (12.7, 45.7), turned to 180 degrees
- moved T1 42.2 mm to (44.5, 88.9), turned to 270 degrees
- moved R3 38.6 mm to (12.7, 48.3), turned to 180 degrees
- moved ANALOG 29.5 mm to (63.5, 91.4)
- moved R5 25.2 mm to (38.1, 87.6), turned to 270 degrees
- moved IC1 24.1 mm to (99.1, 49.5)
- moved R6 16.7 mm to (38.1, 67.3), turned to 270 degrees
- moved U$3 16.5 mm to (19.1, 63.5)
- moved U$2 16.5 mm to (19.1, 83.8)
- moved SW4 16.3 mm to (26.7, 47.0)
- moved POT2 10.2 mm to (53.3, 92.7)
- moved T2 4.58 mm to (44.5, 68.6), turned to 270 degrees
- moved LED1 3.81 mm to (99.1, 10.2)
- moved LED2 3.81 mm to (105.4, 10.2)
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Connections:
- removed net N$2 (its old number): SW4.2, U$2.3
- removed net N$26: R6.P$2, SW4.4
- removed net VCC: IC1.10
- new net GDHJH: R4.P$1, SW4.1
- new net GFHGV: R3.P$1, SW4.2
- new net N$14: IC1.13, Q1.2
- new net N$33: D1.C, IC2.IN
- new net N$35: IC1.12, Q1.1
- new net N$36: IC1.32
- new net N$39: LED9.K, R7.P$1
- new net N$9: D1.A, J2.3, SV1.1
- new net RESET: IC1.9, U$1.5
- net 5V: now also IC1.10, IC2.OUT, LED9.A, PORTA.9, PORTB.9, PORTC.9, PORTD.9, SV1.3, U$1.2
- net A0: now also A.1, PORTA.8; no longer ANALOG1.1
- net A1: now also PORTA.7
- net A2: now also PORTA.6
- net A3: now also PORTA.5
- net A4: now also PORTA.4
- net A5: now also PORTA.3
- net A6: now also PORTA.2
- net A7: now also PORTA.1
- net B0: now also PORTB.8
- net B1: now also PORTB.7
- net B2: now also PORTB.6
- net B3: now also PORTB.5
- net B4: now also PORTB.4
- net B5: now also PORTB.3, U$1.4
- net B6: now also PORTB.2, U$1.1
- net B7: now also PORTB.1, U$1.3
- net C0: now also PORTC.8
- net C1: now also PORTC.7
- net C2: now also PORTC.6
- net C3: now also PORTC.5
- net C4: now also PORTC.4
- net C5: now also PORTC.3
- net C6: now also PORTC.2
- net C7: now also PORTC.1
- net D0: now also PORTD.1, SW4.3; no longer R3.P$1
- net D1: now also PORTD.2, SW4.4; no longer R4.P$1
- net D2: now also PORTD.3
- net D3: now also PORTD.4
- net D4: now also PORTD.5
- net D5: now also PORTD.6
- net D6: now also PORTD.7
- net D7: now also PORTD.8
- net GND: now also IC2.GND, J2.1, J2.2, PORTA.10, PORTB.10, PORTC.10, PORTD.10, R7.P$2, SV1.2, U$1.6
- net N$28: now also U$2.3; no longer SW4.3
- net N$29: now also A.2; no longer ANALOG1.2
- net N$3: now also R6.P$2; no longer SW4.1

Commit message: board
Parts:
- added S17: DTS-3, switch-tact:DTS-3
- moved SW5 18.3 mm to (83.8, 69.8), turned to 0 degrees
- moved S1 6.35 mm to (102.9, 94.0)
- moved S13 6.35 mm to (102.9, 74.9)
- moved S5 6.35 mm to (102.9, 87.6)
- moved S9 6.35 mm to (102.9, 81.3)
- moved S10 3.81 mm to (115.6, 81.3)
- moved S14 3.81 mm to (115.6, 74.9)
- moved S2 3.81 mm to (115.6, 94.0)
- moved S6 3.81 mm to (115.6, 87.6)
- moved S11 1.27 mm to (128.3, 81.3)
- moved S12 1.27 mm to (141.0, 81.3)
- moved S15 1.27 mm to (128.3, 74.9)
- moved S16 1.27 mm to (141.0, 74.9)
- moved S3 1.27 mm to (128.3, 94.0)
- moved S4 1.27 mm to (141.0, 94.0)
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Connections:
- net GND: now also S17.2
- net RESET: now also S17.1
Routing:
- net 5V: track 0.00 -> 433.6 mm, vias 0 -> 6
- net GND: track 0.00 -> 418.7 mm, vias 0 -> 7
- net B6: track 0.00 -> 212.9 mm, vias 0 -> 3
- net D1: track 0.00 -> 207.8 mm, vias 0 -> 2
- net B1: track 0.00 -> 167.1 mm, vias 0 -> 3
- net B0: track 0.00 -> 160.9 mm, vias 0 -> 5
- net B5: track 0.00 -> 152.7 mm, vias 0 -> 4
- net D0: track 0.00 -> 151.5 mm, vias 0 -> 2
- net D2: track 0.00 -> 131.1 mm, vias 0 -> 4
- net B4: track 0.00 -> 122.9 mm, vias 0 -> 2
- net B3: track 0.00 -> 121.9 mm, vias 0 -> 4
- net B2: track 0.00 -> 118.6 mm, vias 0 -> 4
- net B7: track 0.00 -> 105.7 mm, vias 0 -> 2
- net N$57: track 0.00 -> 99.8 mm, vias 0 -> 4
- net N$14: track 0.00 -> 99.4 mm, vias 0 -> 2
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- added copper zone on layer 16, net GND
- added copper zone on layer 16, net N$26
- added copper zone on layer 1, net N$37
Other:
- board text added: "1/8/2018"
- board text added: "12V"
- board text added: "5V"
- board text added: "7SEG"
- board text added: "A0"
- board text added: "A0-POT"
- board text added: "ANALOG"
- board text added: "BL"
- board text added: "BY / SROUR for HTI summer training"
- board text added: "GND"
- board text added: "KEYPAD"
- board text added: "LCD"
- board text added: "PORTA"
- board text added: "PORTB"
- board text added: "PORTC"
- board text added: "PORTD"
- board text added: "POWER"
- board text added: "RESET"
