File: eagle/sch.sch (EAGLE design)
At the start: 12 parts, among them IC1 MEGA32-P

Commit message: 2nd
Parts:
- added BACK_LIGHT: (no value), special:SW_DIP-1
- added J1: (no value), SparkFun-Connectors:CONN_16LONGPADS
- added LCD1: LCD-16X2SILK, SparkFun-Displays:LCD-16X2SILK
- added SW2: (no value), special:SW_DIP-8
- added SW3: (no value), special:SW_DIP-4
- added U$1: AVR_SPI_PRG_6PTH, SparkFun:AVR_SPI_PRG_6PTH
- added VR1: 10k, SparkFun-Resistors:TRIMPOT-PTH-10MM-KNOB-1/2W-10%
Connections:
- new net 5V: BACK_LIGHT.2, SW3.5
- new net C0: IC1.(SCL)PC0
- new net C1: IC1.(SDA)PC1
- new net C2: IC1.(TCK)PC2
- new net C3: IC1.(TMS)PC3
- new net C4: IC1.(TDO)PC4
- new net C5: IC1.(TDI)PC5
- new net C6: IC1.(TOSC1)PC6
- new net C7: IC1.(TOSC2)PC7
- new net D0: IC1.(RXD)PD0, SW1.16, SW3.8
- new net D1: IC1.(TXD)PD1, SW1.15, SW3.7
- new net D2: IC1.(INT0)PD2, SW1.14, SW3.6
- new net D3: IC1.(INT1)PD3, SW1.13
- new net D4: IC1.(OC1B)PD4, SW1.12
- new net D5: IC1.(OC1A)PD5, SW1.11
- new net D6: IC1.(ICP)PD6, SW1.10
- new net D7: IC1.(OC2)PD7, SW1.9
- new net LD0: J1.7, LCD1.DB0, SW2.1
- new net LD1: J1.8, LCD1.DB1, SW2.2
- new net LD2: J1.9, LCD1.DB2, SW2.3
- new net LD3: J1.10, LCD1.DB3, SW2.4
- new net LD4: J1.11, LCD1.DB4, SW2.5
- new net LD5: J1.12, LCD1.DB5, SW2.6
- new net LD6: J1.13, LCD1.DB6, SW2.7
- new net LD7: J1.14, LCD1.DB7, SW2.8
- new net N$25: BACK_LIGHT.1, J1.15, LCD1.A
- new net N$4: J1.3, LCD1.VO
- new net N$5: J1.4, LCD1.RS, SW3.3
- new net N$6: J1.5, LCD1.R/W, SW3.2
- new net N$7: J1.6, LCD1.E, SW3.1
- new net RRR: J1.2, LCD1.VDD, SW3.4
- net B0: now also SW2.16; no longer SW1.16
- net B1: now also SW2.15; no longer SW1.15
- net B2: now also SW2.14; no longer SW1.14
- net B3: now also SW2.13; no longer SW1.13
- net B4: now also SW2.12; no longer SW1.12
- net B5: now also SW2.11; no longer SW1.11
- net B6: now also SW2.10; no longer SW1.10
- net B7: now also SW2.9; no longer SW1.9
- net GND: now also J1.1, J1.16, LCD1.K, LCD1.VSS
Other:
- moved on the sheet: LED1, LED2, LED3, LED4, LED5, LED6, LED7, LED8, R1, R2, SW1

Commit message: lcd+7seg
Parts:
- removed VR1: 10k, SparkFun-Resistors:TRIMPOT-PTH-10MM-KNOB-1/2W-10%
- added POT1: (no value), pot:TRIM_EU-B25P
- added R3, R4, R5, R6: 10M, SparkFun-Resistors:10MOHM-HORIZ-1/4W-5%
- added SW4: (no value), SparkFun:SW_DIP-2
- added T1, T2: 2N2222, adafruit:2N2222
- added U$2, U$3: YSD-160AB3C-8, SparkFun-LED:7-SEGMENT-1DIGIT-1INCH-BLUE-EZ
- LED1, LED2, LED3, LED4, LED5, LED6, LED7, LED8: device adafruit:LED5MM -> led:LED5MM
- R1, R2: value 330 -> 10M
Connections:
- new net N$10: R5.1, T1.E
- new net N$11: R6.1, T2.E
- new net N$13: U$3.DP
- new net N$15: U$3.G2
- new net N$16: R4.2, T2.B
- new net N$2: SW4.2, U$2.G1
- new net N$26: R6.2, SW4.4
- new net N$28: R5.2, SW4.3
- new net N$3: SW4.1, U$3.G1
- new net N$32: U$2.DP
- new net N$33: U$2.G2
- new net POT1: J1.3, LCD1.VO, POT1.S
- net 5V: now also POT1.E, T1.C, T2.C
- net B0: now also U$2.A, U$3.A
- net B1: now also U$2.B, U$3.B
- net B2: now also U$2.C, U$3.C
- net B3: now also U$2.D, U$3.D
- net B4: now also U$2.E, U$3.E
- net B5: now also U$2.F, U$3.F
- net B6: now also U$2.G, U$3.G
- net D0: now also R3.1
- net D1: now also R4.1
- net GND: now also POT1.A
- net N$4: now also R3.2, T1.B; no longer J1.3, LCD1.VO
Other:
- moved on the sheet: BACK_LIGHT, J1, LCD1, SW2, SW3, U$1

Commit message: keypad
Parts:
- added S1, S10, S11, S12, S13, S14, S15, S16, S2, S3, S4, S5, S6, S7, S8, S9: DTS-3, switch-tact:DTS-3
- added SW5: (no value), special:SW_DIP-8
Connections:
- new net A0: IC1.(ADC0)PA0, SW5.8
- new net A1: IC1.(ADC1)PA1, SW5.7
- new net A2: IC1.(ADC2)PA2, SW5.6
- new net A3: IC1.(ADC3)PA3, SW5.5
- new net A4: IC1.(ADC4)PA4, SW5.4
- new net A5: IC1.(ADC5)PA5, SW5.3
- new net A6: IC1.(ADC6)PA6, SW5.2
- new net A7: IC1.(ADC7)PA7, SW5.1
- new net N$12: S1.2, S13.2, S5.2, S9.2, SW5.13
- new net N$27: S10.2, S14.2, S2.2, S6.2, SW5.14
- new net N$30: S11.2, S15.2, S3.2, S7.2, SW5.15
- new net N$31: S1.1, S2.1, S3.1, S4.1, SW5.9
- new net N$34: S12.2, S16.2, S4.2, S8.2, SW5.16
- new net N$41: S5.1, S6.1, S7.1, S8.1, SW5.10
- new net N$49: S10.1, S11.1, S12.1, S9.1, SW5.11
- new net N$57: S13.1, S14.1, S15.1, S16.1, SW5.12

Commit message: ADC
Parts:
- added ANALOG, ANALOG1: (no value), special:SW_DIP-1
- added POT2: (no value), pot:TRIM_EU-B25P
Connections:
- new net AVCC: ANALOG.1, IC1.AVCC
- new net N$29: ANALOG1.2, POT2.S
- net 5V: now also ANALOG.2, POT2.E
- net A0: now also ANALOG1.1
- net GND: now also POT2.A
Changed lines of the file:
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@@
 <part name="S15" library="switch-tact" deviceset="DTS-3" device=""/>
 <part name="S16" library="switch-tact" deviceset="DTS-3" device=""/>
+<part name="ANALOG" library="special" library_urn="urn:adsk.eagle:library:367" deviceset="SW_DIP-1" device="" package3d_urn="urn:adsk.eagle:package:26661/1"/>
+<part name="POT2" library="pot" deviceset="TRIM_EU-" device="B25P"/>
+<part name="ANALOG1" library="special" library_urn="urn:adsk.eagle:library:367" deviceset="SW_DIP-1" device="" package3d_urn="urn:adsk.eagle:package:26661/1"/>
 </parts>
 <sheets>
@@
 <instance part="S15" gate="G$1" x="-121.92" y="58.42" rot="R270"/>
 <instance part="S16" gate="G$1" x="-106.68" y="58.42" rot="R270"/>
+<instance part="ANALOG" gate="G$1" x="-50.8" y="170.18"/>
+<instance part="POT2" gate="1" x="-68.58" y="154.94"/>
+<instance part="ANALOG1" gate="G$1" x="-50.8" y="154.94"/>
 </instances>
 <busses>
@@
 <label x="152.4" y="68.58" size="1.778" layer="95"/>
 </segment>
+<segment>
+<pinref part="POT2" gate="1" pin="A"/>
+<junction x="-68.58" y="149.86"/>
+<label x="-68.58" y="144.78" size="1.778" layer="95"/>
+</segment>
 </net>
 <net name="D0" class="0">
@@
 <label x="195.58" y="-33.02" size="1.778" layer="95"/>
 </segment>
+<segment>
+<pinref part="ANALOG" gate="G$1" pin="2"/>
+<junction x="-58.42" y="170.18"/>
+<label x="-68.58" y="170.18" size="1.778" layer="95"/>
+</segment>
+<segment>
+<pinref part="POT2" gate="1" pin="E"/>
+<junction x="-68.58" y="160.02"/>
+<label x="-68.58" y="162.56" size="1.778" layer="95"/>
+</segment>
 </net>
 <net name="C0" class="0">
@@
 <junction x="-43.18" y="91.44"/>
 <label x="-38.1" y="91.44" size="1.778" layer="95"/>
+</segment>
+<segment>
+<pinref part="ANALOG1" gate="G$1" pin="1"/>
+<junction x="-43.18" y="154.94"/>
+<label x="-38.1" y="154.94" size="1.778" layer="95"/>
 </segment>
 </net>
@@
 </segment>
 </net>
+<net name="AVCC" class="0">
+<segment>
+<pinref part="IC1" gate="G$1" pin="AVCC"/>
+<junction x="7.62" y="68.58"/>
+<label x="0" y="68.58" size="1.778" layer="95"/>
+</segment>
+<segment>
+<pinref part="ANALOG" gate="G$1" pin="1"/>
+<junction x="-43.18" y="170.18"/>
+<label x="-38.1" y="170.18" size="1.778" layer="95"/>
+</segment>
+</net>
+<net name="N$29" class="0">
+<segment>
+<pinref part="POT2" gate="1" pin="S"/>
+<junction x="-63.5" y="154.94"/>
+<pinref part="ANALOG1" gate="G$1" pin="2"/>
+<junction x="-58.42" y="154.94"/>
+<wire x1="-63.5" y1="154.94" x2="-58.42" y2="154.94" width="0.1524" layer="91"/>
+</segment>
+</net>

Commit message: sch_001
Parts:
- added D1: 1N4446, diode:1N4446
- added IC2: (no value), v-reg:78MXXL
- added J2: (no value), con-jack:JACK-PLUG0
- added LED9: (no value), led:LED5MM
- added PORTA, PORTB, PORTC, PORTD: (no value), con-lstb:MA10-1
- added Q1: (no value), crystal:CRYTALHC49U-V
- added R7: 10M, SparkFun-Resistors:10MOHM-HORIZ-1/4W-5%
- added SV1: (no value), con-lstb:MA03-1
- renumbered ANALOG1 to A
Connections:
- removed net N$2 (its old number): SW4.2, U$2.G1
- removed net N$26: R6.2, SW4.4
- new net GDHJH: R4.1, SW4.1
- new net GFHGV: R3.1, SW4.2
- new net N$14: IC1.XTAL1, Q1.2
- new net N$33: D1.C, IC2.IN
- new net N$35: IC1.XTAL2, Q1.1
- new net N$36: IC1.AREF
- new net N$39: LED9.C, R7.1
- new net N$9: D1.A, J2.3, SV1.1
- new net RESET: IC1.RESET, U$1.5
- net 5V: now also IC1.VCC, IC2.OUT, LED9.A, PORTA.9, PORTB.9, PORTC.9, PORTD.9, SV1.3, U$1.2
- net A0: now also PORTA.8
- net A1: now also PORTA.7
- net A2: now also PORTA.6
- net A3: now also PORTA.5
- net A4: now also PORTA.4
- net A5: now also PORTA.3
- net A6: now also PORTA.2
- net A7: now also PORTA.1
- net B0: now also PORTB.8
- net B1: now also PORTB.7
- net B2: now also PORTB.6
- net B3: now also PORTB.5
- net B4: now also PORTB.4
- net B5: now also PORTB.3, U$1.4
- net B6: now also PORTB.2, U$1.1
- net B7: now also PORTB.1, U$1.3
- net C0: now also PORTC.8
- net C1: now also PORTC.7
- net C2: now also PORTC.6
- net C3: now also PORTC.5
- net C4: now also PORTC.4
- net C5: now also PORTC.3
- net C6: now also PORTC.2
- net C7: now also PORTC.1
- net D0: now also PORTD.1, SW4.3; no longer R3.1
- net D1: now also PORTD.2, SW4.4; no longer R4.1
- net D2: now also PORTD.3
- net D3: now also PORTD.4
- net D4: now also PORTD.5
- net D5: now also PORTD.6
- net D6: now also PORTD.7
- net D7: now also PORTD.8
- net GND: now also IC2.GND, J2.1, J2.2, PORTA.10, PORTB.10, PORTC.10, PORTD.10, R7.2, SV1.2, U$1.6
- net N$28: now also U$2.G1; no longer SW4.3
- net N$3: now also R6.2; no longer SW4.1
Other:
- moved on the sheet: R3, R4, R5, R6, SW4, T1, T2, U$1

Commit message: board
Parts:
- added S17: DTS-3, switch-tact:DTS-3
Connections:
- net GND: now also S17.2
- net RESET: now also S17.1
Changed lines of the file:
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@@
 <part name="PORTC" library="con-lstb" library_urn="urn:adsk.eagle:library:162" deviceset="MA10-1" device="" package3d_urn="urn:adsk.eagle:package:8346/1"/>
 <part name="PORTD" library="con-lstb" library_urn="urn:adsk.eagle:library:162" deviceset="MA10-1" device="" package3d_urn="urn:adsk.eagle:package:8346/1"/>
+<part name="S17" library="switch-tact" deviceset="DTS-3" device=""/>
 </parts>
 <sheets>
@@
 <instance part="PORTC" gate="1" x="45.72" y="-48.26" rot="MR90"/>
 <instance part="PORTD" gate="1" x="76.2" y="-48.26" rot="MR90"/>
+<instance part="S17" gate="G$1" x="27.94" y="101.6" rot="R270"/>
 </instances>
 <busses>
@@
 <junction x="-38.1" y="-45.72"/>
 <label x="-38.1" y="-38.1" size="1.778" layer="95" rot="R90"/>
+</segment>
+<segment>
+<pinref part="S17" gate="G$1" pin="2"/>
+<junction x="33.02" y="101.6"/>
+<label x="38.1" y="101.6" size="1.778" layer="95"/>
 </segment>
 </net>
@@
 <junction x="7.62" y="88.9"/>
 <label x="0" y="88.9" size="1.778" layer="95"/>
-</segment>
-</net>
+<pinref part="S17" gate="G$1" pin="1"/>
+<junction x="22.86" y="101.6"/>
+<wire x1="22.86" y1="101.6" x2="7.62" y2="101.6" width="0.1524" layer="91"/>
+<wire x1="7.62" y1="101.6" x2="7.62" y2="88.9" width="0.1524" layer="91"/>
+</segment>
+</net>
